Commit message: 补充夹爪末端TCP草案

File: workspace/ubuntu/carm_ws/src/carm_a3_description/urdf/carm_a3.urdf (robot description, URDF)
Before this commit: robot carm_a3, 11 links, 10 joints
Links:
- added link gripper_tcp
Joints:
- added joint gripper_base_to_tcp: type fixed, parent gripper_base, child gripper_tcp, origin xyz=0 0 0.149 rpy=0 0 0

Commit message: 根据整机模型更新夹爪TCP草案

File: workspace/ubuntu/carm_ws/src/carm_a3_description/urdf/carm_a3.urdf (robot description, URDF)
Before this commit: robot carm_a3, 12 links, 11 joints
Joints:
- joint joint6_to_gripper_base: origin xyz=0 0 0 rpy=0 0 0 -> xyz=0.064891 0.005939 -0.035486 rpy=3.141592654 -0.002999991 3.141592654; parent link6 -> flange

Commit message: 修正夹爪TCP方向并启用抓取补偿

File: workspace/ubuntu/carm_ws/src/carm_a3_description/urdf/carm_a3.urdf (robot description, URDF)
Before this commit: robot carm_a3, 12 links, 11 joints
Joints:
- joint gripper_base_to_tcp: origin xyz=0 0 0.149 rpy=0 0 0 -> xyz=0 0 -0.149 rpy=0 0 0

Commit message: 按夹指模型重定义抓取TCP

File: workspace/ubuntu/carm_ws/src/carm_a3_description/urdf/carm_a3.urdf (robot description, URDF)
Before this commit: robot carm_a3, 12 links, 11 joints
Joints:
- joint gripper_base_to_tcp: origin xyz=0 0 -0.149 rpy=0 0 0 -> xyz=0 0 0.1105 rpy=0 0 0

Commit message: 恢复抓取TCP方向并增加安全高度阶段

File: workspace/ubuntu/carm_ws/src/carm_a3_description/urdf/carm_a3.urdf (robot description, URDF)
Before this commit: robot carm_a3, 12 links, 11 joints
Joints:
- joint gripper_base_to_tcp: origin xyz=0 0 0.1105 rpy=0 0 0 -> xyz=0 0 -0.149 rpy=0 0 0
